File: hardware/digital.kicad_pcb (KiCad board)
At the start: 4 copper layers, 489 parts, among them J1 BNC, J10 Conn_01x03_Pin, J11 Conn_01x03_Pin, J12 Conn_01x10_Pin, J13 Conn_01x02_Pin, J14 Conn_01x03_Pin, J15 Conn_01x02_Pin, J16 Conn_01x03_Pin, J17 Micro_SD_Card_Det1, J18 Conn_01x03_Pin, J19 Micro_SD_Card_Det1, J2 BNC, J20 USB_C_Receptacle_USB2.0_16P, J21 USB_C_Receptacle_USB2.0_16P, J22 USB_C_Receptacle_USB2.0_16P, J23 IPX, J24 IPX, J25 IPX, J26 IPX, J27 IPX, J28 IPX, J29 IPX, J3 BNC, J30 IPX, J31 Conn_01x08_Pin, J32 Conn_01x03_Pin, J33 Conn_01x08_Pin, J34 Conn_01x08_Pin, J35 IPX, J36 IPX, J37 IPX, J38 IPX, J39 IPX, J4 BNC, J40 IPX, J41 IPX, J42 IPX, J43 IPX, J44 IPX, J45 IPX, J46 IPX, J47 IPX, J48 IPX, J49 IPX, J5 BNC, J50 IPX, J51 IPX, J52 IPX, J53 IPX, J54 IPX, J55 IPX, J56 IPX, J57 IPX, J58 IPX, J6 BNC, J7 BNC, J8 BNC, J9 BNC, Q1 BSC098N10NS5, Q2 BSC098N10NS5, SW1 SW_DIP_x03, SW2 SW_DIP_x03, SW3 SW_DIP_x03, SW4 SW_DIP_x03, SW5 SW_DIP_x03, SW6 SW_DIP_x03, SW7 SW_DIP_x03, U1 ICE40HX4K-TQ144, U10 LM5050-1, U11 CH224K, U12 LM5050-1, U13 CH224K, U14 TPS54302, U15 TPS7A7002DDA, U16 TPS54302, U17 TPS7A7002DDA, U18 74HC244, U19 74HC244, U2 74HC244, U20 74HC244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

Commit message: route power
Parts:
- moved C72 303.7 mm to (126.4, 221.9)
- moved C73 303.7 mm to (108.6, 212.5)
- moved C74 303.7 mm to (126.4, 223.8)
- moved C75 303.7 mm to (126.4, 225.8)
- moved C76 303.7 mm to (126.9, 212.1)
- moved C77 303.7 mm to (126.9, 214.6)
- moved C78 303.7 mm to (108.6, 215.9)
- moved C79 303.7 mm to (126.4, 227.8)
- moved C80 303.7 mm to (108.6, 219.2)
- moved C81 303.7 mm to (126.4, 229.7)
- moved C82 303.7 mm to (113.6, 212.3)
- moved C83 303.7 mm to (113.6, 215.3)
- moved C84 303.7 mm to (113.6, 218.4)
- moved C85 303.7 mm to (129.2, 221.9)
- moved C86 303.7 mm to (108.6, 222.6)
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
Commit message: route more
Parts:
- removed J13: Conn_01x02_Pin, Connector_PinHeader_2.54mm:PinHeader_1x02_P2.54mm_Vertical
- added C147: 100n, Capacitor_SMD:C_0402_1005Metric, F.Cu at (138.5, 97.5)
- added C148: 100n, Capacitor_SMD:C_0402_1005Metric, F.Cu at (141.2, 101.4)
- added TP17: TestPoint_Alt, digital:TestPoint_Keystone_5015_Micro_Mini, F.Cu at (149.2, -2.50)
- added TP18: TestPoint_Alt, digital:TestPoint_Keystone_5015_Micro_Mini, F.Cu at (222.0, 103.7)
- added TP19: TestPoint_Alt, digital:TestPoint_Keystone_5015_Micro_Mini, F.Cu at (139.0, 126.0)
- added TP20: TestPoint_Alt, digital:TestPoint_Keystone_5015_Micro_Mini, F.Cu at (149.0, 137.0)
- added TP21: TestPoint_Alt, digital:TestPoint_Keystone_5015_Micro_Mini, F.Cu at (152.0, 137.0)
- added TP22: TestPoint_Alt, digital:TestPoint_Keystone_5015_Micro_Mini, F.Cu at (163.0, 140.0)
- added TP23: TestPoint_Alt, digital:TestPoint_Keystone_5015_Micro_Mini, F.Cu at (167.0, 140.0)
- added TP24: TestPoint_Alt, digital:TestPoint_Keystone_5015_Micro_Mini, F.Cu at (179.0, 136.0)
- added TP25: TestPoint_Alt, digital:TestPoint_Keystone_5015_Micro_Mini, F.Cu at (182.0, 136.0)
- added TP26: TestPoint_Alt, digital:TestPoint_Keystone_5015_Micro_Mini, F.Cu at (191.0, 127.6)
- added TP27: TestPoint_Alt, digital:TestPoint_Keystone_5015_Micro_Mini, F.Cu at (191.0, 125.0)
- added TP28: TestPoint_Alt, digital:TestPoint_Keystone_5015_Micro_Mini, F.Cu at (201.0, 116.0)
- added TP29: TestPoint_Alt, digital:TestPoint_Keystone_5015_Micro_Mini, F.Cu at (202.0, 113.0)
- added TP30: TestPoint_Alt, digital:TestPoint_Keystone_5015_Micro_Mini, F.Cu at (203.0, 102.0)
- added TP31: TestPoint_Alt, digital:TestPoint_Keystone_5015_Micro_Mini, F.Cu at (202.0, 98.0)
- added TP32: TestPoint_Alt, digital:TestPoint_Keystone_5015_Micro_Mini, F.Cu at (201.0, 86.0)
- added TP33: TestPoint_Alt, digital:TestPoint_Keystone_5015_Micro_Mini, F.Cu at (200.0, 83.0)
- added TP34: TestPoint_Alt, digital:TestPoint_Keystone_5015_Micro_Mini, F.Cu at (193.0, 73.0)
- added TP35: TestPoint_Alt, digital:TestPoint_Keystone_5015_Micro_Mini, F.Cu at (190.0, 72.0)
- added TP36: TestPoint_Alt, digital:TestPoint_Keystone_5015_Micro_Mini, F.Cu at (181.0, 64.0)
- added TP37: TestPoint_Alt, digital:TestPoint_Keystone_5015_Micro_Mini, F.Cu at (178.0, 63.0)
- added TP38: TestPoint_Alt, digital:TestPoint_Keystone_5015_Micro_Mini, F.Cu at (167.0, 62.0)
- added TP39: TestPoint_Alt, digital:TestPoint_Keystone_5015_Micro_Mini, F.Cu at (163.0, 62.0)
- added TP40: TestPoint_Alt, digital:TestPoint_Keystone_5015_Micro_Mini, F.Cu at (152.0, 65.0)
- added TP41: TestPoint_Alt, digital:TestPoint_Keystone_5015_Micro_Mini, F.Cu at (148.0, 65.0)
- added TP42: TestPoint_Alt, digital:TestPoint_Keystone_5015_Micro_Mini, F.Cu at (138.0, 72.0)
- added TP43: TestPoint, TestPoint:TestPoint_Pad_D1.0mm, B.Cu at (137.5, 99.9)
- added TP44: TestPoint, TestPoint:TestPoint_Pad_D1.0mm, B.Cu at (137.5, 97.9)
- J1, J3, J6, J7, J8, J9: footprint digital:BNC_TEConnectivity_1478204_Vertical -> digital:DOSIN-801-0078
- J10, J11, J14, J16, J32: footprint Connector_PinHeader_2.54mm:PinHeader_1x03_P2.54mm_Vertical -> Connector_PinHeader_1.00mm:PinHeader_1x03_P1.00mm_Vertical_SMD_Pin1Left; moved to B.Cu
- J12: footprint Connector_PinHeader_2.54mm:PinHeader_1x10_P2.54mm_Vertical -> Connector_PinHeader_1.00mm:PinHeader_1x10_P1.00mm_Vertical_SMD_Pin1Left; moved to B.Cu
- J15: footprint Connector_PinHeader_2.54mm:PinHeader_1x02_P2.54mm_Vertical -> Connector_PinHeader_1.00mm:PinHeader_1x02_P1.00mm_Vertical_SMD_Pin1Left; moved to B.Cu
- J18: footprint Connector_PinHeader_2.54mm:PinHeader_1x03_P2.54mm_Vertical -> Connector_PinHeader_1.00mm:PinHeader_1x03_P1.00mm_Vertical_SMD_Pin1Left
- J2, J4, J5: value BNC -> IPEX-1; footprint digital:BNC_TEConnectivity_1478204_Vertical -> digital:BWIPX-1-001E
- J23, J24, J25, J26, J27, J28, J29, J30, J35, J36, J37, J38, J39, J40, J41, J42, J43, J44, J45, J46, J47, J48, J49, J50, J51, J52, J53, J54, J55, J56, J57, J58: value IPX -> IPEX-1
- J31, J33, J34: footprint Connector_PinHeader_2.54mm:PinHeader_1x08_P2.54mm_Vertical -> Connector_PinHeader_1.00mm:PinHeader_1x08_P1.00mm_Vertical_SMD_Pin1Left; moved to B.Cu
- TP10, TP12, TP13, TP2, TP3, TP5, TP6, TP9: moved to B.Cu
- TP16: value TestPoint -> TestPoint_Alt; footprint TestPoint:TestPoint_Pad_D1.0mm -> digital:TestPoint_Keystone_5015_Micro_Mini
- moved R85 299.8 mm to (128.4, 70.9), turned to 90 degrees
- moved C6 299.7 mm to (170.6, 195.5)
- moved D1 299.7 mm to (186.1, 161.3)
- moved D4 299.7 mm to (186.1, 170.5)
- moved D9 299.7 mm to (186.1, 182.6)
- moved C13 299.7 mm to (191.1, 164.8)
- moved C17 299.7 mm to (191.1, 171.5)
- moved C20 299.7 mm to (191.1, 174.9)
- moved D2 299.7 mm to (186.1, 164.4)
- moved D3 299.7 mm to (186.1, 167.4)
- moved D5 299.7 mm to (186.1, 173.5)
- moved D6 299.7 mm to (186.1, 176.5)
- moved D7 299.7 mm to (170.5, 198.5)
- moved D8 299.7 mm to (186.1, 179.6)
- moved R20 299.7 mm to (161.5, 195.4)
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Connections:
- C12 pad 1: +1V2 -> +3V3
- C9 pad 1: +1V2 -> +3V3
- TP16 pad 1: Net-(SW7-Pad4) -> /dac/VREF_B
Routing:
- net Net-(U13-VDD): track 0.00 -> 23.6 mm, vias 0 -> 5
- net Net-(U11-VDD): track 0.00 -> 23.6 mm, vias 0 -> 5
- net Net-(U13-CFG3): track 0.00 -> 17.5 mm, vias 0 -> 2
- net Net-(U11-CFG3): track 0.00 -> 17.5 mm, vias 0 -> 2
- net Net-(U13-CFG2): track 0.00 -> 16.9 mm, vias 0 -> 2
- net Net-(U11-CFG2): track 0.00 -> 16.9 mm, vias 0 -> 2
- net Net-(J22-CC1): track 0.00 -> 14.0 mm
- net Net-(J20-CC1): track 0.00 -> 14.0 mm
- net Net-(U11-DP): track 0.00 -> 12.0 mm
- net Net-(U13-DP): track 0.00 -> 11.9 mm
- net Net-(J20-CC2): track 0.00 -> 11.6 mm
- net Net-(J22-CC2): track 0.00 -> 11.6 mm
- net Net-(U13-CFG1): track 0.00 -> 9.71 mm, vias 0 -> 2
- net Net-(U11-CFG1): track 0.00 -> 9.70 mm, vias 0 -> 2
- net Net-(U13-DM): track 0.00 -> 7.62 mm
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
Commit message: route mcu
Parts:
- added C149: 100n, Capacitor_SMD:C_0402_1005Metric, F.Cu at (125.5, 113.5)
- J1, J3, J6, J7, J8, J9: value BNC -> IPEX-1; footprint digital:DOSIN-801-0078 -> digital:BWIPX-1-001E
- J18: footprint Connector_PinHeader_1.00mm:PinHeader_1x03_P1.00mm_Vertical_SMD_Pin1Left -> Connector_PinHeader_2.54mm:PinHeader_1x03_P2.54mm_Vertical
- moved C98 269.8 mm to (130.0, 65.2), turned to -90 degrees
- moved R34 266.5 mm to (111.5, 109.2)
- moved R31 263.7 mm to (111.5, 105.8)
- moved C100 261.1 mm to (121.0, 65.4), turned to -90 degrees
- moved C101 254.4 mm to (121.0, 67.9), turned to 180 degrees
- moved C102 252.3 mm to (112.0, 65.4), turned to -90 degrees
- moved C99 249.4 mm to (130.0, 67.9), turned to 180 degrees
- moved C103 245.9 mm to (112.0, 67.9), turned to 180 degrees
- moved J17 209.5 mm to (6.00, 119.0), turned to -90 degrees
- moved R33 199.3 mm to (16.8, 112.0), turned to 90 degrees
- moved C33 195.9 mm to (16.3, 122.5)
- moved R32 192.9 mm to (15.8, 112.0), turned to -90 degrees
- moved R22 187.7 mm to (22.8, 87.1), turned to 90 degrees
- moved C35 187.3 mm to (16.2, 104.0)
- moved R29 187.2 mm to (30.8, 82.5), turned to 180 degrees
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Connections:
- net Net-(J18-Pin_1) renamed /MCU/SWCLK
- net Net-(J18-Pin_3) renamed /MCU/SWD
- net Net-(U4-USB_DM) renamed /MCU/D-
- net Net-(U4-USB_DP) renamed /MCU/D+
Routing:
- net +3V3: track 29.6 -> 84.6 mm
- net +1V2: track 0.00 -> 13.9 mm
- net Net-(J11-Pin_3): track 0.00 -> 13.0 mm, vias 0 -> 1
- net /MCU/QSPI_SS: track 0.00 -> 12.4 mm
- net /MCU/QSPI_SD1: track 0.00 -> 11.1 mm
- net /MCU/QSPI_SD3: track 0.00 -> 10.4 mm
- net Net-(J11-Pin_2): track 0.00 -> 10.2 mm, vias 0 -> 1
- net Net-(J11-Pin_1): track 0.00 -> 10.2 mm, vias 0 -> 1
- net /MCU/XIN: track 0.00 -> 9.64 mm
- net /MCU/QSPI_SD2: track 0.00 -> 9.42 mm
- net /MCU/QSPI_SCLK: track 0.00 -> 8.91 mm
- net Net-(J16-Pin_2): track 0.00 -> 8.88 mm, vias 0 -> 1
- net Net-(J14-Pin_3): track 0.00 -> 8.44 mm, vias 0 -> 1
- net Net-(J10-Pin_3): track 0.00 -> 8.29 mm, vias 0 -> 1
- net Net-(J16-Pin_3): track 0.00 -> 8.09 mm, vias 0 -> 1
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
Commit message: wire until sipm power
Parts:
- removed J31, J33, J34: Conn_01x08_Pin, Connector_PinHeader_1.00mm:PinHeader_1x08_P1.00mm_Vertical_SMD_Pin1Left
- removed J32: Conn_01x03_Pin, Connector_PinHeader_1.00mm:PinHeader_1x03_P1.00mm_Vertical_SMD_Pin1Left
- A1, TP1: moved to B.Cu
- R20: footprint Resistor_SMD:R_0603_1608Metric -> Resistor_SMD:R_0402_1005Metric
- moved R103 185.0 mm to (5.60, 54.8), turned to -90 degrees
- moved A1 172.5 mm to (-8.11, 47.1), turned to 180 degrees
- moved C92 162.2 mm to (54.5, 83.8), turned to 90 degrees
- moved C94 157.6 mm to (64.1, 86.3), turned to 180 degrees
- moved TP17 155.3 mm to (82.0, 137.5), turned to -90 degrees
- moved R83 155.1 mm to (64.6, 81.4), turned to 180 degrees
- moved C142 154.8 mm to (97.0, 143.1)
- moved SW7 154.8 mm to (90.0, 140.0)
- moved C91 152.7 mm to (52.8, 83.8), turned to 90 degrees
- moved U16 151.8 mm to (64.8, 92.4)
- moved C93 151.5 mm to (67.3, 83.5), turned to 90 degrees
- moved U17 150.4 mm to (59.1, 83.5)
- moved C88 150.3 mm to (68.3, 88.4), turned to 90 degrees
- moved R79 148.0 mm to (64.6, 84.4)
- moved C87 147.9 mm to (61.4, 92.4), turned to -90 degrees
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Connections:
- A1 pad D1: Net-(A1-SWCLK) -> unconnected-(A1-SWCLK-PadD1)
- A1 pad D3: Net-(A1-SWDIO) -> unconnected-(A1-SWDIO-PadD3)
Routing:
- net Net-(U1E-GNDPLL0): track 7.74 -> 30.4 mm
- net Net-(U1E-VCCPLL0): track 4.82 -> 27.4 mm
- net Net-(J11-Pin_3): track 13.0 -> 0.00 mm, vias 1 -> 0
- net Net-(J11-Pin_2): track 10.2 -> 0.00 mm, vias 1 -> 0
- net Net-(J11-Pin_1): track 10.2 -> 0.00 mm, vias 1 -> 0
- net +6V_B: track 0.00 -> 9.71 mm
- net +6V_A: track 0.00 -> 9.71 mm
- net Net-(U14-EN): track 0.00 -> 8.55 mm
- net Net-(U16-EN): track 0.00 -> 8.39 mm
- net Net-(J10-Pin_3): track 8.29 -> 0.00 mm, vias 1 -> 0
- net Net-(U5-EN): track 0.00 -> 8.13 mm
- net Net-(U5-FB): track 0.00 -> 8.11 mm
- net Net-(U8-EN): track 0.00 -> 8.09 mm
- net Net-(U9-EN): track 0.00 -> 8.01 mm
- net Net-(U16-FB): track 0.00 -> 7.90 mm
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Other:
- board outline added: 186.7 x 100 mm
