File: hardware/mcu.kicad_sch (KiCad schematic)
At the start: 42 parts, among them J17 Micro_SD_Card_Det1, J18 Conn_01x03_Pin, J19 Micro_SD_Card_Det1, U3 W25Q32JVZP, U4 RP2040, Y1 12 MHz ABM8-272-T3

Commit message: route
Parts:
- renumbered C21 to C24, C22 to C25, C23 to C26, C24 to C27, C25 to C28, C26 to C29, C27 to C30, C28 to C31, C29 to C32, C30 to C33, C31 to C34, C32 to C35, C33 to C36, C34 to C37, C35 to C38, C36 to C39, C37 to C40, J17 to J16, J18 to J17, J19 to J18
Connections:
- net ~{LDAC}0: now also U4.9 (GPIO7); no longer U4.4 (GPIO2)
- net ~{LDAC}1: now also U4.8 (GPIO6); no longer U4.5 (GPIO3)
- net ~{LDAC}2: now also U4.7 (GPIO5); no longer U4.6 (GPIO4)
- net ~{LDAC}3: now also U4.6 (GPIO4); no longer U4.7 (GPIO5)
- net ~{LDAC}4: now also U4.5 (GPIO3); no longer U4.8 (GPIO6)
- net ~{LDAC}5: now also U4.4 (GPIO2); no longer U4.9 (GPIO7)
Changed lines of the file:
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@@
 		)
 	)
+	(label "~{LDAC}3"
+		(at 128.27 78.74 180)
+		(effects
+			(font
+				(size 1.27 1.27)
+			)
+			(justify right bottom)
+		)
+	)
 	(label "DET_A"
 		(at 198.12 113.03 0)
@@
 		)
 	)
-	(label "~{LDAC}5"
-		(at 128.27 86.36 180)
-		(effects
-			(font
-				(size 1.27 1.27)
-			)
-			(justify right bottom)
-		)
-	)
 	(label "DET_B"
 		(at 128.27 144.78 180)
@@
 		)
 	)
-	(label "~{LDAC}1"
-		(at 128.27 76.2 180)
-		(effects
-			(font
-				(size 1.27 1.27)
-			)
-			(justify right bottom)
-		)
-	)
 	(label "QSPI_SD2"
 		(at 220.98 50.8 0)
@@
 		)
 	)
-	(label "QSPI_SD2"
-		(at 57.15 96.52 0)
+	(label "~{LDAC}4"
+		(at 128.27 76.2 180)
 		(effects
 			(font
 				(size 1.27 1.27)
 			)
-			(justify left bottom)
+			(justify right bottom)
 		)
 	)
-	(label "QSPI_SD3"
-		(at 57.15 99.06 0)
+	(label "QSPI_SD2"
+		(at 57.15 96.52 0)
 		(effects
 			(font
@@
 		)
 	)
-	(label "~{LDAC}2"
-		(at 128.27 78.74 180)
+	(label "QSPI_SD3"
+		(at 57.15 99.06 0)
 		(effects
 			(font
 				(size 1.27 1.27)
 			)
-			(justify right bottom)
+			(justify left bottom)
 		)
 	)
@@
 		)
 	)
+	(label "~{LDAC}0"
+		(at 128.27 86.36 180)
+		(effects
+			(font
+				(size 1.27 1.27)
+			)
+			(justify right bottom)
+		)
+	)
 	(label "CS_B"
 		(at 215.9 132.08 0)
@@
 		)
 	)
-	(label "CS_A"
-		(at 215.9 92.71 0)
+	(label "~{LDAC}1"
+		(at 128.27 83.82 180)
 		(effects
 			(font
 				(size 1.27 1.27)
 			)
-			(justify left bottom)
+			(justify right bottom)
 		)
 	)
-	(label "SD_SO"
-		(at 215.9 105.41 0)
+	(label "CS_A"
+		(at 215.9 92.71 0)
 		(effects
 			(font
@@
 		)
 	)
-	(label "~{LDAC}4"
-		(at 128.27 83.82 180)
+	(label "SD_SO"
+		(at 215.9 105.41 0)
 		(effects
 			(font
 				(size 1.27 1.27)
 			)
-			(justify right bottom)
+			(justify left bottom)
 		)
 	)
@@
 		)
 	)
+	(label "~{LDAC}2"
+		(at 128.27 81.28 180)
+		(effects
+			(font
+				(size 1.27 1.27)
+			)
+			(justify right bottom)
+		)
+	)
 	(label "DET_B"
 		(at 198.12 152.4 0)
@@
 		)
 	)
-	(label "~{LDAC}0"
+	(label "~{LDAC}5"
 		(at 128.27 73.66 180)
 		(effects
@@
 		)
 	)
-	(label "~{LDAC}3"
-		(at 128.27 81.28 180)
-		(effects
-			(font
-				(size 1.27 1.27)
-			)
-			(justify right bottom)
-		)
-	)
 	(label "XIN"
 		(at 57.15 114.3 0)
@@
 		(on_board yes)
 		(dnp no)
-		(property "Reference" "C23"
+		(property "Reference" "C26"
 			(at 113.284 29.718 0)
 			(effects
@@
 			(project "digital"
 				(path "/4c5c7ce5-09d6-4a32-b2a0-f32b0c47f27d/7712deab-3fc2-4c53-b3e8-8bdddd2adcec"
-					(reference "C23")
+					(reference "C26")
 					(unit 1)
 				)
@@
 		(dnp no)
 		(fields_autoplaced yes)
-		(property "Reference" "J17"
+		(property "Reference" "J16"
 			(at 253.365 78.74 0)
 			(effects
@@
 			(project ""
 				(path "/4c5c7ce5-09d6-4a32-b2a0-f32b0c47f27d/7712deab-3fc2-4c53-b3e8-8bdddd2adcec"
-					(reference "J17")
+					(reference "J16")
 					(unit 1)
 				)
@@
 		(on_board yes)
 		(dnp no)
-		(property "Reference" "C22"
+		(property "Reference" "C25"
 			(at 78.994 29.718 0)
 			(effects
@@
 			(project "digital"
 				(path "/4c5c7ce5-09d6-4a32-b2a0-f32b0c47f27d/7712deab-3fc2-4c53-b3e8-8bdddd2adcec"
-					(reference "C22")
+					(reference "C25")
 					(unit 1)
 				)
@@
 		(on_board yes)
 		(dnp no)
-		(property "Reference" "C24"
+		(property "Reference" "C27"
 			(at 123.444 29.718 0)
 			(effects
@@
 			(project "digital"
 				(path "/4c5c7ce5-09d6-4a32-b2a0-f32b0c47f27d/7712deab-3fc2-4c53-b3e8-8bdddd2adcec"
-					(reference "C24")
+					(reference "C27")
 					(unit 1)
 				)
@@
 		(on_board yes)
 		(dnp no)
-		(property "Reference" "C25"
+		(property "Reference" "C28"
 			(at 132.334 29.718 0)
 			(effects
@@
 			(project "digital"
 				(path "/4c5c7ce5-09d6-4a32-b2a0-f32b0c47f27d/7712deab-3fc2-4c53-b3e8-8bdddd2adcec"
-					(reference "C25")
+					(reference "C28")
 					(unit 1)
 				)
@@
 		(on_board yes)
 		(dnp no)
-		(property "Reference" "C36"
+		(property "Reference" "C39"
 			(at 36.068 168.91 90)
 			(effects
@@
 			(project "digital"
 				(path "/4c5c7ce5-09d6-4a32-b2a0-f32b0c47f27d/7712deab-3fc2-4c53-b3e8-8bdddd2adcec"
-					(reference "C36")
+					(reference "C39")
 					(unit 1)
 				)
@@
 		(on_board yes)
 		(dnp no)
-		(property "Reference" "C34"
+		(property "Reference" "C37"
 			(at 189.992 138.1759 0)
 			(effects
@@
 			(project "digital"
 				(path "/4c5c7ce5-09d6-4a32-b2a0-f32b0c47f27d/7712deab-3fc2-4c53-b3e8-8bdddd2adcec"
-					(reference "C34")
+					(reference "C37")
 					(unit 1)
 				)
@@
 		(on_board yes)
 		(dnp no)
-		(property "Reference" "C33"
+		(property "Reference" "C36"
 			(at 196.342 98.8059 0)
 			(effects
@@
 			(project "digital"
 				(path "/4c5c7ce5-09d6-4a32-b2a0-f32b0c47f27d/7712deab-3fc2-4c53-b3e8-8bdddd2adcec"
-					(reference "C33")
+					(reference "C36")
 					(unit 1)
 				)
@@
 		(on_board yes)
 		(dnp no)
-		(property "Reference" "C26"
+		(property "Reference" "C29"
 			(at 141.224 29.718 0)
 			(effects
@@
 			(project "digital"
 				(path "/4c5c7ce5-09d6-4a32-b2a0-f32b0c47f27d/7712deab-3fc2-4c53-b3e8-8bdddd2adcec"
-					(reference "C26")
+					(reference "C29")
 					(unit 1)
 				)
@@
 		(on_board yes)
 		(dnp no)
-		(property "Reference" "J18"
+		(property "Reference" "J17"
 			(at 39.116 133.858 0)
 			(effects
@@
 			(project "digital"
 				(path "/4c5c7ce5-09d6-4a32-b2a0-f32b0c47f27d/7712deab-3fc2-4c53-b3e8-8bdddd2adcec"
-					(reference "J18")
+					(reference "J17")
 					(unit 1)
 				)
@@
 		(on_board yes)
 		(dnp no)
-		(property "Reference" "C27"
+		(property "Reference" "C30"
 			(at 150.114 29.718 0)
 			(effects
@@
 			(project "digital"
 				(path "/4c5c7ce5-09d6-4a32-b2a0-f32b0c47f27d/7712deab-3fc2-4c53-b3e8-8bdddd2adcec"
-					(reference "C27")
+					(reference "C30")
 					(unit 1)
 				)
@@
 		(on_board yes)
 		(dnp no)
-		(property "Reference" "C21"
+		(property "Reference" "C24"
 			(at 68.834 29.718 0)
 			(effects
@@
 			(project "digital"
 				(path "/4c5c7ce5-09d6-4a32-b2a0-f32b0c47f27d/7712deab-3fc2-4c53-b3e8-8bdddd2adcec"
-					(reference "C21")
+					(reference "C24")
 					(unit 1)
 				)
@@
 		(on_board yes)
 		(dnp no)
-		(property "Reference" "C30"
+		(property "Reference" "C33"
 			(at 78.994 44.958 0)
 			(effects
@@
 			(project "digital"
 				(path "/4c5c7ce5-09d6-4a32-b2a0-f32b0c47f27d/7712deab-3fc2-4c53-b3e8-8bdddd2adcec"
-					(reference "C30")
+					(reference "C33")
 					(unit 1)
 				)
@@
 		(on_board yes)
 		(dnp no)
-		(property "Reference" "C28"
+		(property "Reference" "C31"
 			(at 159.004 29.718 0)
 			(effects
@@
 			(project "digital"
 				(path "/4c5c7ce5-09d6-4a32-b2a0-f32b0c47f27d/7712deab-3fc2-4c53-b3e8-8bdddd2adcec"
-					(reference "C28")
+					(reference "C31")
 					(unit 1)
 				)
@@
 		(on_board yes)
 		(dnp no)
-		(property "Reference" "C29"
+		(property "Reference" "C32"
 			(at 268.986 33.528 0)
 			(effects
@@
 			(project "digital"
 				(path "/4c5c7ce5-09d6-4a32-b2a0-f32b0c47f27d/7712deab-3fc2-4c53-b3e8-8bdddd2adcec"
-					(reference "C29")
+					(reference "C32")
 					(unit 1)
 				)
@@
 		(on_board yes)
 		(dnp no)
-		(property "Reference" "C37"
+		(property "Reference" "C40"
 			(at 36.068 184.15 90)
 			(effects
@@
 			(project "digital"
 				(path "/4c5c7ce5-09d6-4a32-b2a0-f32b0c47f27d/7712deab-3fc2-4c53-b3e8-8bdddd2adcec"
-					(reference "C37")
+					(reference "C40")
 					(unit 1)
 				)
@@
 		(on_board yes)
 		(dnp no)
-		(property "Reference" "C35"
+		(property "Reference" "C38"
 			(at 196.342 138.1759 0)
 			(effects
@@
 			(project "digital"
 				(path "/4c5c7ce5-09d6-4a32-b2a0-f32b0c47f27d/7712deab-3fc2-4c53-b3e8-8bdddd2adcec"
-					(reference "C35")
+					(reference "C38")
 					(unit 1)
 				)
@@
 		(dnp no)
 		(fields_autoplaced yes)
-		(property "Reference" "J19"
+		(property "Reference" "J18"
 			(at 253.365 118.11 0)
 			(effects
@@
 			(project "digital"
 				(path "/4c5c7ce5-09d6-4a32-b2a0-f32b0c47f27d/7712deab-3fc2-4c53-b3e8-8bdddd2adcec"
-					(reference "J19")
+					(reference "J18")
 					(unit 1)
 				)
@@
 		(on_board yes)
 		(dnp no)
-		(property "Reference" "C31"
+		(property "Reference" "C34"
 			(at 113.284 44.958 0)
 			(effects
@@
 			(project "digital"
 				(path "/4c5c7ce5-09d6-4a32-b2a0-f32b0c47f27d/7712deab-3fc2-4c53-b3e8-8bdddd2adcec"
-					(reference "C31")
+					(reference "C34")
 					(unit 1)
 				)
@@
 		(on_board yes)
 		(dnp no)
-		(property "Reference" "C32"
+		(property "Reference" "C35"
 			(at 189.992 98.8059 0)
 			(effects
@@
 			(project "digital"
 				(path "/4c5c7ce5-09d6-4a32-b2a0-f32b0c47f27d/7712deab-3fc2-4c53-b3e8-8bdddd2adcec"
-					(reference "C32")
+					(reference "C35")
 					(unit 1)
 				)
