File: hardware/digital.kicad_sch (KiCad schematic)
At the start: 18 parts, among them J1 IPEX-1, J2 IPEX-1, J3 IPEX-1, J4 IPEX-1, J5 IPEX-1, J6 IPEX-1, J7 IPEX-1, J8 IPEX-1, J9 IPEX-1

Commit message: finish pcb
Parts:
- added H1, H2, H3, H4, H5, H6: M4, MountingHole:MountingHole_4.3mm_M4_ISO14580_Pad_TopBottom, symbol Mechanical:MountingHole_Pad
Connections:
- net GND: now also H1.1, H2.1, H3.1, H4.1, H5.1, H6.1

Commit message: fabrication
Parts:
- R1, R2: LCSC C17168 -> C25120
Changed lines of the file:
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@@
 			)
 		)
-		(property "LCSC" "C17168"
+		(property "LCSC" "C25120"
 			(at 104.14 91.44 0)
 			(effects
@@
 			)
 		)
-		(property "LCSC" "C17168"
+		(property "LCSC" "C25120"
 			(at 104.14 93.98 0)
 			(effects
